Commit message: feat: add dual-arm perception and manipulation workflow

File: agibot_x2_moveit_config/config/x2_ultra.ros2_control.xacro (robot description, xacro)
@@ -40,6 +40,6 @@
           <param name="arm_command_topic">/aima/hal/joint/arm/command</param>
           <param name="zmq_endpoint">${zmq_endpoint}</param>
-          <param name="state_timeout_sec">0.1</param>
-          <param name="activation_timeout_sec">2.0</param>
+          <param name="state_timeout_sec">0.25</param>
+          <param name="activation_timeout_sec">10.0</param>
           <param name="fault_damping">5.0</param>
           <param name="fault_publish_duration_sec">0.2</param>

File: agibot_x2_moveit_config/config/x2_ultra.urdf.xacro (robot description, xacro)
@@ -6,6 +6,36 @@
     <xacro:arg name="command_transport" default="ros_topic" />
     <xacro:arg name="zmq_endpoint" default="tcp://*:8559" />
+    <xacro:arg name="left_hand_pad_origin" default="0 0 -0.13" />
+    <xacro:arg name="right_hand_pad_origin" default="0 0 -0.13" />
+    <xacro:property name="hand_pad_thickness" value="0.012" />
+    <xacro:property name="hand_pad_width" value="0.08" />
+    <xacro:property name="hand_pad_height" value="0.10" />
     <!-- Import x2_ultra urdf file -->
     <xacro:include filename="$(find x2_description)/urdf/x2_ultra.urdf" />
+    <!-- Passive pads: left TCP -Y and right TCP +Y pass through the contact surface. -->
+    <xacro:macro name="x2_hand_pad" params="side origin tcp_y">
+      <link name="${side}_hand_pad_link">
+        <visual>
+          <geometry><box size="${hand_pad_width} ${hand_pad_thickness} ${hand_pad_height}"/></geometry>
+          <material name="x2_contact_pad"><color rgba="0.15 0.15 0.15 1"/></material>
+        </visual>
+        <collision><geometry><box size="${hand_pad_width} ${hand_pad_thickness} ${hand_pad_height}"/></geometry></collision>
+        <inertial>
+          <mass value="0.05"/><origin xyz="0 0 0"/>
+          <inertia ixx="0.0000417" ixy="0" ixz="0" iyy="0.0000417" iyz="0" izz="0.0000417"/>
+        </inertial>
+      </link>
+      <joint name="${side}_hand_pad_joint" type="fixed">
+        <parent link="${side}_wrist_roll_link"/><child link="${side}_hand_pad_link"/>
+        <origin xyz="${origin}" rpy="0 0 0"/>
+      </joint>
+      <link name="${side}_hand_tcp_link"/>
+      <joint name="${side}_hand_tcp_joint" type="fixed">
+        <parent link="${side}_hand_pad_link"/><child link="${side}_hand_tcp_link"/>
+        <origin xyz="0 ${tcp_y} 0" rpy="0 0 0"/>
+      </joint>
+    </xacro:macro>
+    <xacro:x2_hand_pad side="left" origin="$(arg left_hand_pad_origin)" tcp_y="${-hand_pad_thickness / 2.0}"/>
+    <xacro:x2_hand_pad side="right" origin="$(arg right_hand_pad_origin)" tcp_y="${hand_pad_thickness / 2.0}"/>
     <!-- Import control_xacro -->
     <xacro:include filename="x2_ultra.ros2_control.xacro" />
